File: hardware/vegas26-badge/vegas26-badge.kicad_sch (KiCad schematic)
At the start: 38 parts, among them J1 RAW_EPD_FPC_24, J2 AUDIO_PIGTAIL, J3 TC2050_IDC_NL_DNL, J4 ESP_RIBBON_1x08_P2.54_DNP, Q1 BSS138

Commit message: new badge
Other:
- title: AISB Vegas 2026 Raw E-Paper Badge -> AISB 2026 Raw E-Paper Badge
Changed lines of the file:
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@@
 	(paper "A4")
 	(title_block
-		(title "AISB Vegas 2026 Raw E-Paper Badge")
+		(title "AISB 2026 Raw E-Paper Badge")
 		(date "2026-07-15")
 		(rev "2")
