File: hardware/aisb/aisb.kicad_pcb (KiCad board)
At the start: 2 copper layers, 100 x 145 mm, 42 parts, among them J1 FH34SRJ-24S-0.5SH(50)/(99) / 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, J2 AUDIO, J3 TC2050-IDC-NL / DNL, J4 1x08 P2.54 / OPTIONAL / DNP, Q1 BSS138

Commit message: Update badge silkscreen to San Francisco and align initials full stops
Co-Authored-By: Claude Opus 5.5 (1M context) <noreply@anthropic.com>
Other:
- board text added: "AI SECURITY BOOTCAMP · SAN FRANCISCO 2026"
- board text removed: "AI SECURITY BOOTCAMP · LONDON 2026"
Changed lines of the file:
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@@
 		)
 	)
-	(gr_text "AI SECURITY BOOTCAMP · LONDON 2026"
+	(gr_text "AI SECURITY BOOTCAMP · SAN FRANCISCO 2026"
 		(at 49 48 0)
 		(layer "F.SilkS")
